File: hardware/simon-keychain/simon-keychain.kicad_pcb (KiCad board)
At the start: 2 copper layers, 1 part, among them U1 ATtiny85-20SU

Commit message: Schematic updated
Parts:
- added BT1: Battery_Cell, Batteries:BATT_CR2032_MPD, B.Cu at (154.9, 82.5)
- added BZ1: Buzzer, Buzzer_Beeper:Buzzer_CUI_CPT-9019S-SMT, B.Cu at (135.9, 82.5)
- added D1: LED, LED_SMD:LED_1206_3216Metric_Pad1.42x1.75mm_HandSolder, F.Cu at (138.6, 67.3)
- added D2: LED, LED_SMD:LED_1206_3216Metric_Pad1.42x1.75mm_HandSolder, F.Cu at (164.8, 67.3)
- added D3: LED, LED_SMD:LED_1206_3216Metric_Pad1.42x1.75mm_HandSolder, F.Cu at (144.4, 99.1)
- added D4: LED, LED_SMD:LED_1206_3216Metric_Pad1.42x1.75mm_HandSolder, F.Cu at (163.8, 99.1)
- added R1: R, Resistor_SMD:R_0805_2012Metric_Pad1.15x1.40mm_HandSolder, F.Cu at (149.9, 80.0)
- added R2: R, Resistor_SMD:R_0805_2012Metric_Pad1.15x1.40mm_HandSolder, F.Cu at (149.9, 83.0)
- added R3: R, Resistor_SMD:R_0805_2012Metric_Pad1.15x1.40mm_HandSolder, F.Cu at (154.6, 80.0)
- added R4: R, Resistor_SMD:R_0805_2012Metric_Pad1.15x1.40mm_HandSolder, F.Cu at (154.6, 83.0)
- added R5: R, Resistor_SMD:R_0805_2012Metric_Pad1.15x1.40mm_HandSolder, B.Cu at (132.3, 88.9)
- added SW1: SW_Push, Button_Switch_SMD:SW_Push_1P1T_NO_6x6mm_H9.5mm, F.Cu at (141.0, 91.4)
- added SW2: SW_Push, Button_Switch_SMD:SW_Push_1P1T_NO_6x6mm_H9.5mm, F.Cu at (141.0, 72.4)
- added SW3: SW_Push, Button_Switch_SMD:SW_Push_1P1T_NO_6x6mm_H9.5mm, F.Cu at (161.3, 91.4)
- added SW4: SW_Push, Button_Switch_SMD:SW_Push_1P1T_NO_6x6mm_H9.5mm, F.Cu at (161.3, 72.4)
- U1: moved to B.Cu
- moved U1 1.27 mm to (135.9, 94.0)
Connections:
- U1 pad 4: Net-(U1-Pad4) -> GND
- U1 pad 8: Net-(U1-Pad8) -> +3V3

Commit message: update
Parts:
- added C1: C, Capacitor_SMD:C_0805_2012Metric_Pad1.15x1.40mm_HandSolder, B.Cu at (142.0, 75.7)
- added REF**: MountingHole_2.2mm_M2_Pad_Via, MountingHole:MountingHole_2.2mm_M2_Pad_Via, F.Cu at (136.1, 66.7)
- BT1: footprint Batteries:BATT_CR2032_MPD -> Battery:BatteryHolder_Keystone_1058_1x2032
- BZ1: moved to F.Cu
- R1, R2, R3, R4: moved to B.Cu
- moved R3 19.4 mm to (139.7, 92.5), turned to 270 degrees
- moved SW1 18.8 mm to (142.7, 72.7)
- moved SW2 17.5 mm to (142.4, 89.8)
- moved R5 17.4 mm to (138.2, 72.5), turned to 270 degrees
- moved BZ1 16.7 mm to (152.6, 81.3), turned to 45 degrees
- moved R4 15.1 mm to (145.2, 71.1)
- moved D4 15.1 mm to (163.2, 83.9)
- moved D3 14.7 mm to (142.5, 84.5)
- moved U1 12.7 mm to (139.7, 81.9), turned to 90 degrees
- moved R2 12.2 mm to (155.2, 94.0)
- moved R1 11.8 mm to (140.8, 72.5), turned to 90 degrees
- moved D1 11.6 mm to (142.5, 78.2)
- moved D2 10.5 mm to (163.5, 77.7)
- moved SW3 2.16 mm to (162.5, 89.6)
- moved BT1 1.51 mm to (155.2, 81.1), turned to 45 degrees
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Other:
- board outline added: 37.2 x 32.3 mm

Commit message: PCB rooted
Parts:
- added G***: LOGO, Symbol:Github_logo, F.Cu at (142.9, 94.8)
- added J1: AVR-ISP-6, Connector_PinHeader_2.54mm:PinHeader_2x03_P2.54mm_Vertical_SMD_ISP, B.Cu at (164.1, 92.2)
- added SW5: SW_SPDT, Button_Switch_SMD:SW_SPDT_PCM12, B.Cu at (146.4, 68.2)
- BZ1: footprint Buzzer_Beeper:Buzzer_CUI_CPT-9019S-SMT -> Buzzer_Beeper:PUIAudio_SMT_0825_S_4_R
- SW1, SW2, SW3, SW4: footprint Button_Switch_SMD:SW_Push_1P1T_NO_6x6mm_H9.5mm -> Button_Switch_SMD:SW_SPST_PTS645
- moved R4 22.6 mm to (137.7, 92.4), turned to 90 degrees
- moved R5 2.45 mm to (139.6, 70.5), turned to 180 degrees
- moved R1 2.41 mm to (139.0, 74.1), turned to 180 degrees
- moved R2 1.13 mm to (154.1, 94.1)
- moved D2 0.94 mm to (162.8, 78.2), turned to 180 degrees
- moved C1 0.46 mm to (142.4, 75.8)
- moved D4 0.45 mm to (162.8, 84.0), turned to 180 degrees
- moved R3 0.26 mm to (140.0, 92.4), turned to 90 degrees
- moved BT1 0.23 mm to (155.4, 81.0), turned to 225 degrees
Connections:
- net Net-(R1-Pad2) renamed MISO
- net Net-(R2-Pad2) renamed SCK
- net Net-(R5-Pad2) renamed MOSI
- BT1 pad 1: +3V3 -> Net-(BT1-Pad1)
- U1 pad 1: Net-(U1-Pad1) -> RST
Routing:
- net SCK: track 0.00 -> 72.5 mm, vias 0 -> 2
- net MISO: track 0.00 -> 66.2 mm, vias 0 -> 1
- net +3V3: track 0.00 -> 59.6 mm, vias 0 -> 1
- net MOSI: track 0.00 -> 46.3 mm
- net Net-(D4-Pad1): track 0.00 -> 43.6 mm, vias 0 -> 1
- net Net-(D2-Pad1): track 0.00 -> 37.0 mm, vias 0 -> 1
- net RST: track 0.00 -> 25.9 mm
- net Net-(R4-Pad2): track 0.00 -> 25.8 mm, vias 0 -> 1
- net Net-(BT1-Pad1): track 0.00 -> 21.6 mm
- net Net-(R3-Pad2): track 0.00 -> 21.5 mm, vias 0 -> 1
- net Net-(D1-Pad1): track 0.00 -> 21.5 mm, vias 0 -> 1
- net Net-(BZ1-Pad1): track 0.00 -> 18.5 mm, vias 0 -> 1
- net Net-(D3-Pad1): track 0.00 -> 18.1 mm, vias 0 -> 1
- net GND: vias 0 -> 1
- added copper zone on B.Cu, net GND
- added copper zone on F.Cu, net GND
Other:
- board size 37.2 x 32.3 mm -> 36 x 32.3 mm
- board text added: "Galco6/simon-keychain"

Commit message: Updated PCB
Parts:
- added G***: LOGO, Symbol:OSHW-Logo_3x3mm_SilkScreen, B.Cu at (165.9, 85.9)
Changed lines of the file:
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@@
   (general
     (thickness 1.6)
-    (drawings 15)
+    (drawings 13)
     (tracks 165)
     (zones 0)
-    (modules 21)
+    (modules 22)
     (nets 18)
   )
@@
     (add_net SCK)
   )
+  (module Symbol:OSHW-Logo_3x3mm_SilkScreen (layer B.Cu)
+    (at 165.9255 85.852 180)
+    (fp_text reference G*** (at 0 0) (layer B.SilkS) hide
+      (effects (font (size 1.524 1.524) (thickness 0.3)) (justify mirror))
+    )
+    (fp_text value LOGO (at 0.75 0) (layer B.SilkS) hide
+      (effects (font (size 1.524 1.524) (thickness 0.3)) (justify mirror))
+    )
+    (fp_poly (pts (xy 0.175773 1.63545) (xy 0.218141 1.61867) (xy 0.242742 1.581571) (xy 0.259011 1.516303)
+      (xy 0.27638 1.415017) (xy 0.277503 1.408545) (xy 0.29788 1.300912) (xy 0.319275 1.228203)
+      (xy 0.349313 1.179634) (xy 0.395619 1.144423) (xy 0.465815 1.111787) (xy 0.495963 1.099568)
+      (xy 0.649511 1.038099) (xy 0.834596 1.165595) (xy 0.915287 1.220107) (xy 0.981719 1.262987)
+      (xy 1.024845 1.288502) (xy 1.035779 1.293091) (xy 1.057894 1.277704) (xy 1.104391 1.236288)
+      (xy 1.167496 1.17596) (xy 1.2117 1.132032) (xy 1.371525 0.970973) (xy 1.106755 0.585165)
+      (xy 1.178212 0.425899) (xy 1.213553 0.348454) (xy 1.241692 0.289231) (xy 1.257349 0.259295)
+      (xy 1.258395 0.257909) (xy 1.283709 0.249738) (xy 1.342539 0.236186) (xy 1.422935 0.21997)
+      (xy 1.435969 0.217504) (xy 1.550689 0.1967) (xy 1.628051 0.180194) (xy 1.675327 0.160397)
+      (xy 1.699784 0.12972) (xy 1.708693 0.080576) (xy 1.709321 0.005375) (xy 1.708728 -0.067242)
+      (xy 1.706792 -0.181981) (xy 1.700496 -0.256471) (xy 1.689107 -0.296503) (xy 1.678379 -0.306887)
+      (xy 1.641957 -0.316017) (xy 1.573633 -0.329432) (xy 1.487159 -0.344463) (xy 1.47328 -0.346723)
+      (xy 1.386757 -0.36205) (xy 1.317813 -0.376792) (xy 1.27941 -0.388126) (xy 1.276864 -0.389502)
+      (xy 1.258995 -0.416452) (xy 1.231182 -0.473498) (xy 1.198993 -0.547237) (xy 1.167999 -0.624267)
+      (xy 1.143767 -0.691185) (xy 1.131866 -0.734589) (xy 1.131455 -0.739458) (xy 1.143901 -0.767577)
+      (xy 1.17723 -0.823431) (xy 1.225427 -0.897214) (xy 1.251985 -0.935986) (xy 1.372515 -1.10936)
+      (xy 1.20741 -1.274464) (xy 1.042306 -1.439569) (xy 0.858869 -1.31914) (xy 0.675433 -1.19871)
+      (xy 0.590352 -1.239283) (xy 0.557059 -1.255665) (xy 0.531286 -1.265038) (xy 0.509448 -1.262458)
+      (xy 0.487959 -1.242981) (xy 0.463236 -1.201662) (xy 0.431692 -1.133557) (xy 0.389744 -1.033723)
+      (xy 0.333806 -0.897215) (xy 0.32272 -0.870184) (xy 0.182308 -0.528095) (xy 0.246773 -0.477639)
+      (xy 0.357326 -0.375572) (xy 0.427224 -0.27064) (xy 0.46153 -0.153457) (xy 0.467147 -0.069273)
+      (xy 0.446396 0.075734) (xy 0.387554 0.19938) (xy 0.295744 0.296602) (xy 0.176085 0.36234)
+      (xy 0.033697 0.391531) (xy 0 0.392545) (xy -0.14668 0.372031) (xy -0.271752 0.313861)
+      (xy -0.370096 0.223097) (xy -0.436593 0.104803) (xy -0.46612 -0.03596) (xy -0.467147 -0.069273)
+      (xy -0.452631 -0.198966) (xy -0.405708 -0.310508) (xy -0.321315 -0.413282) (xy -0.246772 -0.477639)
+      (xy -0.182307 -0.528095) (xy -0.32272 -0.870184) (xy -0.381375 -1.013374) (xy -0.425434 -1.119056)
+      (xy -0.458484 -1.192173) (xy -0.484107 -1.23767) (xy -0.505891 -1.260489) (xy -0.527418 -1.265577)
+      (xy -0.552275 -1.257876) (xy -0.584046 -1.24233) (xy -0.590351 -1.239283) (xy -0.675432 -1.19871)
+      (xy -0.852827 -1.315173) (xy -0.931652 -1.3662) (xy -0.995019 -1.405864) (xy -1.033755 -1.428488)
+      (xy -1.041048 -1.431636) (xy -1.060858 -1.416302) (xy -1.105456 -1.375013) (xy -1.167351 -1.314842)
+      (xy -1.212023 -1.270251) (xy -1.372171 -1.108866) (xy -1.251813 -0.935739) (xy -1.19867 -0.856903)
+      (xy -1.157524 -0.791306) (xy -1.134392 -0.748763) (xy -1.131454 -0.739458) (xy -1.14006 -0.70269)
+      (xy -1.162167 -0.639594) (xy -1.192204 -0.563575) (xy -1.224604 -0.488034) (xy -1.253796 -0.426375)
+      (xy -1.274214 -0.391999) (xy -1.276863 -0.389502) (xy -1.30883 -0.379022) (xy -1.373527 -0.364658)
+      (xy -1.45799 -0.349231) (xy -1.473279 -0.346723) (xy -1.561309 -0.331681) (xy -1.63328 -0.317847)
+      (xy -1.675441 -0.307893) (xy -1.678378 -0.306887) (xy -1.693552 -0.286523) (xy -1.703146 -0.235543)
+      (xy -1.707893 -0.148159) (xy -1.708727 -0.067242) (xy -1.709567 0.030838) (xy -1.707242 0.097522)
+      (xy -1.694481 0.140399) (xy -1.664017 0.167059) (xy -1.608579 0.185089) (xy -1.520899 0.202078)
+      (xy -1.435968 0.217504) (xy -1.353391 0.233883) (xy -1.290607 0.248002) (xy -1.259566 0.257143)
+      (xy -1.258394 0.257909) (xy -1.245402 0.281725) (xy -1.219024 0.336721) (xy -1.184541 0.411833)
+      (xy -1.178212 0.425899) (xy -1.106754 0.585165) (xy -1.371524 0.970973) (xy -1.211699 1.132032)
+      (xy -1.142186 1.200532) (xy -1.084445 1.254549) (xy -1.046249 1.286964) (xy -1.035778 1.293091)
+      (xy -1.011016 1.280774) (xy -0.957509 1.247645) (xy -0.884305 1.199438) (xy -0.834596 1.165595)
+      (xy -0.64951 1.038099) (xy -0.495963 1.099568) (xy -0.41607 1.13375) (xy -0.362619 1.166899)
+      (xy -0.327986 1.209798) (xy -0.304547 1.273229) (xy -0.284678 1.367976) (xy -0.277502 1.408545)
+      (xy -0.259814 1.511943) (xy -0.243722 1.578909) (xy -0.219794 1.617294) (xy -0.178595 1.634947)
+      (xy -0.110692 1.639718) (xy -0.00665 1.639458) (xy 0 1.639454) (xy 0.106204 1.639761)
+      (xy 0.175773 1.63545)) (layer B.SilkS) (width 0.01))
+  )
   (module Button_Switch_SMD:SW_SPDT_PCM12 (layer B.Cu)
     (at 146.3675 68.199)
@@
     )
   )
-  (dimension 32.321501 (width 0.12) (layer F.SilkS)
-    (gr_text "32,322 mm" (at 153.955749 59.690001 1.772683129e-06) (layer F.SilkS)
-      (effects (font (size 1 1) (thickness 0.15)))
-    )
-    (feature1 (pts (xy 170.1165 66.04) (xy 170.1165 60.37358)))
-    (feature2 (pts (xy 137.794999 66.040001) (xy 137.794999 60.373581)))
-    (crossbar (pts (xy 137.794999 60.960002) (xy 170.1165 60.960001)))
-    (arrow1a (pts (xy 170.1165 60.960001) (xy 168.989996 61.546422)))
-    (arrow1b (pts (xy 170.1165 60.960001) (xy 168.989996 60.37358)))
-    (arrow2a (pts (xy 137.794999 60.960002) (xy 138.921503 61.546423)))
-    (arrow2b (pts (xy 137.794999 60.960002) (xy 138.921503 60.373581)))
-  )
-  (dimension 27.305 (width 0.12) (layer F.SilkS)
-    (gr_text "27,305 mm" (at 124.333 82.804 270) (layer F.SilkS)
-      (effects (font (size 1 1) (thickness 0.15)))
-    )
-    (feature1 (pts (xy 135.255 96.4565) (xy 125.016579 96.4565)))
-    (feature2 (pts (xy 135.255 69.1515) (xy 125.016579 69.1515)))
-    (crossbar (pts (xy 125.603 69.1515) (xy 125.603 96.4565)))
-    (arrow1a (pts (xy 125.603 96.4565) (xy 125.016579 95.329996)))
-    (arrow1b (pts (xy 125.603 96.4565) (xy 126.189421 95.329996)))
-    (arrow2a (pts (xy 125.603 69.1515) (xy 125.016579 70.278004)))
-    (arrow2b (pts (xy 125.603 69.1515) (xy 126.189421 70.278004)))
-  )
   (gr_line (start 160.147 81.28) (end 169.037 81.28) (layer F.SilkS) (width 0.12))

Commit message: Updated readme
Other:
- board text added: "Galco6/SimonKeychain"
- board text removed: "Galco6/simon-keychain"
Changed lines of the file:
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@@
     (tags "Surface mounted pin header SMD 2x03 2.54mm double row")
     (attr smd)
-    (fp_text reference J1 (at 0 4.87) (layer B.SilkS)
+    (fp_text reference J1 (at 0 0) (layer B.SilkS)
       (effects (font (size 1 1) (thickness 0.15)) (justify mirror))
     )
@@
     (tags "mounting hole 2.2mm m2")
     (attr virtual)
-    (fp_text reference REF** (at 0 -3.2) (layer F.SilkS)
-      (effects (font (size 1 1) (thickness 0.15)))
-    )
-    (fp_text value MountingHole_2.2mm_M2_Pad_Via (at 0 3.2) (layer F.Fab)
+    (fp_text reference REF** (at 4.2545 1.9685) (layer F.SilkS) hide
+      (effects (font (size 1 1) (thickness 0.15)))
+    )
+    (fp_text value MountingHole_2.2mm_M2_Pad_Via (at 0 3.2) (layer F.Fab) hide
       (effects (font (size 1 1) (thickness 0.15)))
     )
@@
   (gr_line (start 145.4785 81.28) (end 135.8265 81.28) (layer F.SilkS) (width 0.12))
   (gr_line (start 152.5905 74.168) (end 152.5905 66.675) (layer F.SilkS) (width 0.12))
-  (gr_text Galco6/simon-keychain (at 154.3685 94.8055) (layer F.SilkS)
+  (gr_text Galco6/SimonKeychain (at 154.3685 94.8055) (layer F.SilkS)
     (effects (font (size 1 1) (thickness 0.2)))
   )
